Commit message: Update maze and robot to be just like prof asked in the pdf

File: robot.urdf (robot description, URDF)
Before this commit: robot maze_runner, 4 links, 3 joints
Links:
- link base_link: geometry collision cylinder length=0.1 radius=1.0; visual cylinder length=0.1 radius=1.0
Joints:
- joint caster_joint: origin xyz=0.15 0 -0.05 -> xyz=0.8 0 -0.05
- joint left_motor: origin xyz=-0.1 0.175 0 -> xyz=-0.1 1.05 0
- joint right_motor: origin xyz=-0.1 -0.175 0 -> xyz=-0.1 -1.05 0
